Commit message: PR3 — Extendable column (prismatic STS3215 lift on a static mast, closes #73) (#76)
* PR3: extendable column — prismatic STS3215 lift on a static mast

Fills urdf/column.xacro: a static `column_rail_link` mast fixed to
`base_link` at the chassis puck's top surface (computed from base.xacro's
own properties), and a `column_top` carriage riding it on the prismatic
`column_lift`, whose limits are RobotModel's 0.00-1.20 m of travel.
`column_top`'s link frame is the arm/head mount datum; the carriage body
hangs below it. Every dimension is an xacro property marked SOURCED or
ESTIMATED, inertias computed from those properties.

The gate grows by six: the lift is the model's only prismatic joint and is
wired rail -> carriage; its limits equal the transcribed RobotModel bounds;
its effort/velocity are present and positive; its axis is +z after every rpy
above it is composed; the mast clears the chassis and spans the travel its
own carriage is allowed; and the carriage body sits below its mount datum.
Each was confirmed by perturbing the model and watching that test, and only
that test, fail.

Co-Authored-By: Claude Opus 5 <noreply@anthropic.com>

* docs: ratify the column as D31 and flatten it into the current-state docs

D31 records the mast+carriage topology and why the third fixed link was
refused, the prismatic parented to the rail rather than base_link (sibling
contact is filtered nowhere), the mount height computed from the base's own
properties and the include-order coupling that buys, the travel-vs-absolute
semantics of the limits and the residue PR6 must reconcile, and the
transcribed RobotModel constants as a pin PR6 removes. It also records the
contradiction it could not resolve: D26's "~600 mm rail" and RobotModel's
1.20 m of travel cannot both be literal.

spec.md's "Column, arms, grippers, camera and the MJCF are still to come"
became false with this change, which is exactly the failure D30 was filed
for, so it is fixed here rather than in a follow-up.

Co-Authored-By: Claude Opus 5 <noreply@anthropic.com>

* test: route the column's limit reads through one legible guard

A prismatic joint with no <limit> is rejected by check_urdf and by
robot_state_publisher, so the three assertions that read one were reporting
that single root cause as three AttributeErrors on None. `_lift_limit` does
for them what `_require_expansion` already does for the expansion. Same for a
missing <axis>, which URDF silently defaults to (1, 0, 0).

Co-Authored-By: Claude Opus 5 <noreply@anthropic.com>

* docs: implementation notes for the column, and say the overlap is deliberate

The carriage wraps its mast, so the two solids interpenetrate by design --
which is the whole reason the prismatic joint parents to the rail rather than
sitting beside it under base_link. Said in the xacro header, where someone
about to "fix" the overlap will read it.

Co-Authored-By: Claude Opus 5 <noreply@anthropic.com>

* fix(#73 round 1): pin the datum, separate capability from policy

B1/R13 — the datum's height above base_link is *both* joint origins plus q
(0.195 + q), not the rail joint's alone; the rail box is centred, so
column_lift's own origin is -0.585. The wrong formula was prose nothing
executed, so it is now a test:
test_column_datum_rests_on_the_mast_foot_at_the_lower_limit asserts the
carriage rests on the mast's foot at zero travel. Measured: the span test
tolerates sliding that origin by up to the over-travel (+0.05 m); this one
catches +0.02 m.

B2/R14 — column_lift_velocity was 0.15, exactly robot_safety's
velocity.column cap. Those are different quantities: the URDF states
capability, limits.yaml states policy, and policy equal to capability is a
clamp that can never bind. Raised to 0.25 (still ESTIMATED, with the residue
recorded), and gated against a transcribed SAFETY_COLUMN_SPEED_CAP_MPS.

B3/R15 — the MoveIt/MuJoCo filtering claim is demoted from fact to
expectation, unverified until PR7, with the fusestatic caveat named. The
parenting stands on kinematic honesty alone.

N1/N2/N3 — lower/upper are asserted as attributes of the raw expansion (URDF
defaults an omitted lower to 0, which was green); the mast gets the
positive-dimension guard the chassis and carriage already had; and the mast's
visual must match its collision, as theirs already must.

Co-Authored-By: Claude Opus 5 <noreply@anthropic.com>

* docs: correct D31 and the flattened docs against red-team round 1

R13 — the datum height is both joint origins plus q (0.195 + q), corrected in
D31, the roadmap, spec.md, README and status.md R4. R14 — the
capability-vs-policy distinction, the 0.25 m/s estimate and its residue; R10
and context.md Q4 now name the docs/design-only grep that produced their false
premise. R15 — the MoveIt/MuJoCo filtering is an expectation, unverified until
PR7, with fusestatic named; D31's clause-3 headline no longer calls it a
"fact". R16 — "and only that test" is gone and section 5's table is
re-measured (15 of 19 perturbations are single-cause). R17 — the gate grew by
ten, counted from git diff.

N6/N7 — the merge-order graph's (done) markers move to their own line so the
branch anchors sit under PR3/PR4 again (checked by column index); spec.md no
longer claims a head_camera_link that does not exist.

The N+1 sweep found four restatements the rulings did not list: the datum
formula inside a test's failure message, and the filtering claim in a test
docstring, that test's assertion message and the roadmap's PR3 amendment. It
also caught a claim written this round — the new datum test's docstring said
the span test tolerates a 200 mm slide; measured, it tolerates 50 mm.

Co-Authored-By: Claude Opus 5 <noreply@anthropic.com>

* docs: count the helpers from the diff too

Eight, not six. The same class of error R17 was raised for, in the same
table, caught by the same sweep.

Co-Authored-By: Claude Opus 5 <noreply@anthropic.com>

* red-team: round 2 — the fix diff verified by execution, no BLOCKs

Every round-1 BLOCK (B1-B4) and every ruled-in NOTE (N1, N2, N3, N6, N7) is
re-checked by perturbing a scratch copy of the installed share tree and
watching the suite, not by reading the diff: the datum test pins the identity
to a nanometre (span tolerates +0.05, not +0.06 — both docstring numbers
exact), the velocity inequality reds at 0.15 and 0.14 and greens at 0.16, the
lower/upper declaration hole is closed both ways, the degeneracy and mast-
visual guards fire, and the merge-order graph's anchors are back at columns
15 and 23 by index. The N+1 sweep finds no surviving instance of the four
corrected claims, and the implementation's re-measured perturbation table
reproduces row for row.

One new NOTE (N9): the safety-cap pin is one-directional — a cap raised above
capability leaves every package green — routed to the N5 follow-up.

Co-Authored-By: Claude Opus 5 <noreply@anthropic.com>

* test: say which direction the safety-cap copy can drift in

Red-team round 2, N9. The constant's comment claimed drift "makes the
assertion weaker, never wrong". True of the assertion, misleading about the
property it exists to protect: a cap lowered in limits.yaml leaves this
comparing against a stale higher number and the property still holds, but a
cap raised *above* the URDF's capability is the inversion column.xacro calls
worse than the equality this constant was added to catch -- and the test
still passes, because it reads the copy rather than limits.yaml.

Measured by the red-team: with velocity.column at 0.30, robot_description
and robot_safety stay fully green and only robot_brain's prompt-envelope
test objects, to the prompt rather than to the URDF. Nothing closes that
short of reading the cap live, which costs the dependency edge the
transcription exists to avoid; PR6/PR7 are where to revisit the trade.

Comment only -- no assertion changed. Suite green at 799.

Co-Authored-By: Claude Opus 5 <noreply@anthropic.com>

* red-team: round 3 — one BLOCK, the column's lateral placement is ungated

56260fa checks out: comment-only proven by AST identity (byte-identical dump
either side), and its "only robot_brain objects" claim re-measured across all
nine packages rather than the three round 2 covered. One mis-citation (N10):
the comment attributes a ranking to column.xacro that column.xacro does not
make -- phrasing I introduced in round 2's N9.

B5, found by attacking the axis no previous round touched: every x and y in
the column subassembly is ungated. A mast at x = 5.0 m, a carriage riding
0.5 m to the side of its rail, a carriage narrower than the mast it "wraps" --
each passes all 24 tests, with test_column_rail_stands_on_the_chassis green
for a mast standing on nothing. Every column assertion reads a z. Unlike the
base's analogous check, which discloses that it ignores radial separation and
whose x/y are pinned elsewhere, nothing pins the column's.

N+1 not yet satisfied: fix round, then two clean passes.

Co-Authored-By: Claude Opus 5 <noreply@anthropic.com>

* fix(#73 round 3): gate where the column stands, not just how tall it is

B5/R19 — every column assertion read a z, so the mast's height above the deck
was gated and its position over the deck was not, at any of the four places
the column carries a translation. A mast five metres away passed all 24 tests
with test_column_rail_stands_on_the_chassis green, and D31 clause 3's
measured mast/carriage overlap prism was silently falsifiable in x and y.

Two relational clauses, numbers off the model:

- the mast's collision footprint lies within the puck it stands on, using the
  true corner distance hypot(|x| + w/2, |y| + d/2) for an axis-aligned box --
  not hypot(centre) + half-diagonal, which would reject a legal mast near the
  rim. The chassis is asserted centred rather than assumed, since the
  footprint is measured against its centre.
- test_column_carriage_wraps_the_mast: the rail's cross-section, composed
  through the lift joint's origin and the carriage's own shape offset, is
  contained in the carriage's. That is D31 clause 3's claim, finally asserted
  instead of asserted-about.

Verified: all seven of the red-team's perturbations red, each naming its own
clause; a legal off-centre mast (x=0.08) stays green and x=0.13 reds, so the
gate is a relationship and not a pin at zero.

R20/N10 — column.xacro now states the ranking the test comment cites (the
inversion is worse than the equality, and why), so the citation is true after
status.md is deleted at merge; and the comment no longer forecloses a live
cross-check from a third place that depends on both packages.

Both docstrings say what they do not constrain, per the round-3 lesson.

Co-Authored-By: Claude Opus 5 <noreply@anthropic.com>

* docs: the overlap prism is now asserted, and the gate knows x and y

D31 clause 3 cites test_column_carriage_wraps_the_mast instead of a
measurement somebody took once; clause 6 grows to eleven (counted from git
diff) and its enumeration names the footprint and wrap clauses. Clause 6 also
records what round 3 actually found, because the general form outlives the
instance: every column assertion read a z, orientation was gated at all four
of the column's frames and translation at none of them, and a test whose name
claims more than its assertion checks is the bug.

Same correction in the roadmap, spec.md, the README and the xacro header, all
of which restated the prism as measured rather than gated.

implementation.md: counts re-taken from the diff (11 tests, 9 helpers, floor
14 -> 25), the perturbation table extended with round 3's nine lateral cases
including the two that must stay green, and section 7 now hands the next
reviewer my own list of what is still ungated rather than only what is.

Co-Authored-By: Claude Opus 5 <noreply@anthropic.com>

* docs: re-measure the perturbation counts the new test changed

Adding test_column_carriage_wraps_the_mast moved the rotated-lift-origin
perturbation from three failing tests to four, because it shares the
_axis_aligned_joint guard. Both D31 and implementation.md carried the old
number, and D31's single-cause list said "a zeroed limit" when a zeroed
velocity reds two. D31 now names the mechanism (a perturbation that breaks a
frame reds every assertion composing it) rather than a count that goes stale
the next time the gate grows.

Co-Authored-By: Claude Opus 5 <noreply@anthropic.com>

* red-team: round 4 — the lateral gate is tight, clean pass #1 of two

29 perturbations against the 25-test suite, including base.xacro (which no
previous round touched). All eight of round 3's lateral cases now red, each
naming its own clause; negatives, split offsets that compound, a displaced
chassis puck, and a carriage that wraps in x but misses in y are all caught
too. The footprint boundary lands within 0.1 mm of the corner arithmetic on
both the axis (0.116969) and the diagonal (0.076066), which distinguishes the
true box corner from both approximations the comment says it rejected.

The wrap clause's admitted cross-test dependency behaves as admitted: break
the axis test's premise and only the axis test reds, so the pair catches it
between them. D31's re-measured counts (eleven tests, 3/4/7, seven
single-cause) all re-measured rather than credited. N10 resolves properly --
column.xacro states the ranking and its reasoning is correct on the merits.

Two NOTES, both about where knowledge lives: N11 credits one test with a
conjunction it only half asserts; N12 notes two honest caveats recorded only
in implementation.md, which is deleted at merge.

Co-Authored-By: Claude Opus 5 <noreply@anthropic.com>

* docs: keep the gate's known blind spots in the file that survives merge

Red-team round 4, N11 and N12.

N11: column.xacro credited the whole 0.06 x 0.06 x 0.08 m overlap prism to
test_column_carriage_wraps_the_mast. That test pins the cross-section; the
0.08 m of depth follows from the datum and span tests. True of the suite,
mis-attributed to one test -- the same register of error the last two rounds
kept finding, so it gets the same treatment.

N12: two of the four "still ungated" caveats lived only in
docs/features/.../implementation.md, which CI deletes at merge. They now sit
in test_description.py's module docstring, the file a later PR actually
reads. All four are recorded, none is introduced by the column, and each
names a model that is currently self-consistent and wrong -- including the
measured one: a 0.4 m cube bolted to the mast five metres out passes the
whole suite, because every "drawn as it collides" assertion reads
collisions[0] only.

Comments and docstrings only; no assertion changed. Suite green at 800,
robot_description 25 (+0 ok).

Co-Authored-By: Claude Opus 5 <noreply@anthropic.com>

* red-team: round 5 — clean, N+1 satisfied (two consecutive clean passes)

0466fe1 verified: docstring-and-comment-only proven four ways (docstring-
stripped AST, the 77 assert nodes, the function set, the module constants),
since ast.dump() alone would flag a module-docstring edit that means nothing.

N11's re-attribution is not just true but minimal: destroying each half of the
overlap prism separately shows disjoint test sets -- lift joint x=0.5 kills the
cross-section and reds only the wrap clause; sliding the lift origin +-1.4
kills the depth and reds only the datum and span tests. All four N12 caveats
re-derived against the current 25-test suite rather than transcribed.

Two NOTES. N14: the new blind-spot list's item #1 says "tensors" but the gap is
every physical scalar -- 0.001 N of effort, a 1 g mast and a 500 kg carriage
each pass all 25 tests. N13: two prose counts in the durable test file went
stale when the fix rounds changed the facts under them, both introduced by
868a6a5 and missed by three subsequent rounds.

Co-Authored-By: Claude Opus 5 <noreply@anthropic.com>

* docs: take red-team round 5's two count corrections

N13: the module docstring said "Two column assertions exist because a review
round caught the claim they now pin" -- it is four; the footprint and wrap
clauses are exactly that, added after round 3 found that calling the
interpenetration "measured" left every x and y in the column ungated. And
test_column_lift_is_the_models_only_prismatic_joint said "Four faults" at the
top and "All three faults" fourteen lines down; the three listed inline plus
the uniqueness clause's fourth are now named as such.

N14: caveat 1 of the module docstring's blind-spot list named inertia
tensors, but the gap is every physical scalar -- the round measured a 1 g
mast, a 500 kg carriage and an effort of 0.001 N all green. Positivity is
genuinely all this gate knows, and the caveat now says so.

Both are the red-team's own round-5 text applied; comments and docstrings
only, no assertion changed. Suite green at 800, robot_description 25 (+0 ok).

Co-Authored-By: Claude Opus 5 <noreply@anthropic.com>

* chore: remove ephemeral feature docs for i73-pr3-extendable-column

Merge-time cleanup so the docs-clean guard passes.

---------

Co-authored-by: Claude Opus 5 <noreply@anthropic.com>

File: src/robot_description/urdf/column.xacro (robot description, xacro)
@@ -3,7 +3,271 @@
   Extendable column: one linear-rail STS3215 lift, modeled as a single
   prismatic joint (D26).
-  Deliberately empty: PR1 ships the package and the expand/parse gate only.
-  The column links and the prismatic joint land in PR3.
+  Crib status, stated first because it decides what may be cited below: D26
+  names Nori Bot (arXiv 2605.16537) as the crib for this mechanism and marks it
+  **UNVERIFIED until the paper is read** — spec.md and PROJECT.md carry the same
+  flag. Nothing in this repo records a single dimension of that machine beyond
+  D26's "~600 mm linear rail" paraphrase. So Nori Bot is cribbed here as a
+  *concept* — a lead-screw/linear-rail Z lift driven by one STS3215 on the arm
+  bus, no second controller — and **no number below is attributed to it**. The
+  only sourced numbers are the two travel bounds, which come from this repo's
+  own `RobotModel` (D23); everything else is marked ESTIMATED, because a fake
+  citation is worse than an estimate that says it is one (D29).
+  Shape:
+      base_link ──fixed (column_rail_joint)──▶ column_rail_link   [static mast]
+      column_rail_link ──prismatic (column_lift)──▶ column_top    [carriage]
+  Three things about that shape are deliberate and are the ones to argue with:
+  - **The static mast is modeled.** A lift with 1.2 m of travel has a rail that
+    is physically there at every joint value; describing only the carriage
+    yields a block floating a metre in the air with nothing underneath it —
+    invisible to Nav2/MoveIt collision and structurally absent from PR7's MJCF.
+  - **`column_top` is the carriage itself, and its link frame origin IS the
+    arm/head mount datum**: the carriage body hangs *below* that origin (see the
+    <origin> on its visual/collision/inertial), so PR3.5's head camera and PR4's
+    shoulders mount at `column_top`'s own frame without landing inside the
+    carriage solid. The alternative — a `column_carriage_link` plus a massless
+    `column_top` frame fixed to it — is one more link that corresponds to no
+    body, the modelling artifact D29 refused to import from LeKiwi's CAD chain.
+  - **The prismatic joint's parent is the rail, not `base_link`.** Kinematically
+    identical while `column_rail_joint` is fixed. What decides it is that the
+    carriage *wraps* the rail: the two solids below deliberately interpenetrate
+    (a 0.06 × 0.06 × 0.08 m prism at every reachable joint value — gated, not
+    just measured here, though by the suite rather than by one test:
+    test_column_carriage_wraps_the_mast pins the 0.06 × 0.06 cross-section,
+    while the 0.08 m of depth follows from the datum and span tests), which is what
+    a carriage on a mast does, and shaving them apart would describe a
+    mechanism that falls over. Parenting the carriage to the rail it rides is
+    simply the honest kinematic description of that, and it is the
+    arrangement collision tooling is *expected* to filter — MoveIt's generated
+    ACM disables adjacent pairs, MuJoCo excludes parent/child bodies — where
+    two siblings under `base_link` would be filtered by neither.
+    That expectation is **unverified and stays so until PR7 builds the MJCF**:
+    there is no SRDF in this repo (so there is no ACM yet), and a *fixed* rail
+    joint is a strong candidate for MuJoCo's `fusestatic`, which would fuse
+    `column_rail_link` into `base_link`'s body and make the carriage's MuJoCo
+    parent `base_link` either way — in which case the filtering comes from body
+    fusion, not from this parenting. **PR7 should check that rather than
+    inherit it.** The parenting stands on kinematic honesty alone.
+  Recorded contradiction (D31): D26 paraphrases the crib as a "~600 mm linear
+  rail" while `RobotModel` demands **1.20 m of travel**. A single-stage carriage
+  on a 600 mm rail cannot travel 1.20 m, so the two cannot both be literal. The
+  travel bound wins here — it is the number the Mock, the safety layer and the
+  brain already enforce — and the mast is therefore authored *longer* than the
+  travel. Whether the real mechanism is a two-stage/telescoping rail (600 mm of
+  rail, 1.2 m of travel) or the travel bound is optimistic is a question for the
+  Nori paper and for PR6, not something to invent an answer to here.
+  Include-order coupling, stated because it is invisible otherwise: the mount
+  height below is computed from `base.xacro`'s own `chassis_z_offset` /
+  `chassis_height`, so this file only expands when `base.xacro` is included
+  first (robot.urdf.xacro does). Reversing that order fails loudly at expansion
+  ("name 'chassis_z_offset' is not defined"), which the gate already runs.
 -->
 <robot xmlns:xacro="http://www.ros.org/wiki/xacro">
+  <!-- ==================================================================
+       Dimensions. Two sourced numbers (the travel bounds); the rest are
+       honest placeholders, marked as such per property.
+       ================================================================== -->
+  <!-- SOURCED (robot_backends, `mock_world.py`): `RobotModel.min_column_height`
+       and `RobotModel.max_column_height`, the column travel the Mock backend,
+       the safety layer and the brain's prompt already enforce. Deliberately
+       spelled with `RobotModel`'s own field names — not prefixed like every
+       other property here — so PR6, which inverts this correspondence and makes
+       `RobotModel` read the URDF, greps one identifier and finds both ends of
+       it. Metres.
+       These are the carriage's **travel along the rail**, measured from
+       `column_lift`'s own origin: they are not heights above `base_link` and
+       not heights above the floor. The mount datum's height above `base_link`
+       at joint value q is **both** joint origins plus q:
+         column_rail_joint.z + column_lift.origin.z + q
+           = chassis_top + column_carriage_height + (q - min_column_height)
+           = 0.195 + q       ->  0.195 m ... 1.395 m today
+       i.e. at the bottom of the travel the carriage rests on the mast's foot
+       and its top face — the datum — is one carriage-height up. `column_lift`'s
+       own origin is *negative* (-0.585 today) because the rail's box is centred
+       in its link frame, so leaving that term out overstates the datum by more
+       than half a metre; the gate pins the identity in
+       test_column_datum_rests_on_the_mast_foot_at_the_lower_limit.
+       The roadmap's table maps these two fields straight onto the lower/upper
+       limit values with no additive term, so the mount offset is deliberately
+       *not* folded into the limits. Which of the two `RobotModel.column_height`
+       itself means is PR6's to reconcile (D31). -->
+  <xacro:property name="min_column_height" value="0.00"/>
+  <xacro:property name="max_column_height" value="1.20"/>
+  <!-- ESTIMATED: the mast's cross-section, m. An aluminium linear-rail
+       extrusion of roughly this size is what a single-servo lead-screw lift is
+       built on; nothing upstream publishes the profile, and the paper that
+       would (D26's Nori crib) is unread. Square, because there is no evidence
+       for an asymmetric one. -->
+  <xacro:property name="column_rail_width" value="0.06"/>
+  <xacro:property name="column_rail_depth" value="0.06"/>
+  <!-- ESTIMATED: rail left over above the carriage at full extension, m. A
+       carriage flush with the end of its own rail is a mechanism with no hard
+       stop and no room for the lead screw's end bearing. 50 mm is a guess with
+       the right sign. -->
+  <xacro:property name="column_rail_overtravel" value="0.05"/>
+  <!-- ESTIMATED: the carriage / mount plate that rides the rail and carries the
+       arms and the head, m. Wider and deeper than the rail because it wraps it;
+       its height is what separates the mount datum from the rail's own bottom
+       stop, so it is a real dimension rather than decoration. -->
+  <xacro:property name="column_carriage_width" value="0.14"/>
+  <xacro:property name="column_carriage_depth" value="0.10"/>
+  <xacro:property name="column_carriage_height" value="0.08"/>
+  <!-- ESTIMATED: masses, kg. Plausible for an extruded aluminium mast and a
+       printed/machined carriage plate with a nut block on it; nothing upstream
+       publishes them. The inertias below are *computed* from the dimensions
+       above, so retuning one cannot leave a stale tensor behind (D29). -->
+  <xacro:property name="column_rail_mass" value="2.5"/>
+  <xacro:property name="column_carriage_mass" value="0.8"/>
+  <!-- ESTIMATED: `column_lift`'s effort (N) and velocity (m/s) limits. Both are
+       **mandatory** — `check_urdf` and `urdf_parser_py` each refuse to parse a
+       `<limit>` that omits either — so there is no honest option of leaving
+       them out, and no STS3215 stall-torque figure, lead-screw pitch or gear
+       ratio is recorded anywhere in this repo to derive them from. They are
+       therefore placeholders with the right order of magnitude for a lift that
+       must hold two arms and a payload against gravity, owed a real actuator
+       model when PR6/PR7 give the servo one. Deliberately not dressed up as a
+       datasheet number (D29).
+       The velocity is a placeholder with a **constraint on it**, which is why
+       it is not simply the roundest number to hand. A URDF `<limit velocity>`
+       is *capability* — what the mechanism can do, and what MoveIt and
+       `ros2_control` plan and clamp against. `robot_safety`'s
+       `robot_safety/limits.yaml` `velocity.column: 0.15` is *policy* — how fast
+       this robot is allowed to move a lift through the height where hands are.
+       Policy must sit strictly **below** capability or the clamp is vacuous:
+       equal, it can never bind for anything that trusts the URDF; above, it
+       would be a cap the machine cannot reach.
+       Of those two, **the inversion (policy above capability) is the worse
+       one**, and it is worth ranking them rather than listing them. Equality
+       is a guard that has stopped guarding: nothing unsafe is commanded,
+       because the machine's own ceiling happens to sit exactly where policy
+       does. The inversion is a guard that is *wrong about the machine*:
+       whatever reads the cap — a planner, the brain's prompt, a future
+       controller — believes in a speed the lift does not have, so the
+       effective limiter silently becomes an unaudited number in a description
+       package instead of the file whose entire job is safety limits, and a
+       command issued at the permitted speed saturates the actuator and turns
+       into a tracking error at runtime rather than a refusal at the seam.
+       So this number's job is to clear 0.15 m/s with room for policy to be
+       tightened after an incident, and the gate asserts that relationship
+       (see SAFETY_COLUMN_SPEED_CAP_MPS in test_description.py).
+       Note the *height* bounds above are deliberately the opposite: there,
+       policy equals capability (`limits.yaml`'s `column.min/max_height` are
+       0.00/1.20 too), and that is correct — a position clamp's job is to stop
+       at the mechanical stop, not short of it.
+       Residue, since a placeholder that now carries a constraint invites
+       over-reading: 0.25 m/s is still a guess. If a real STS3215 through a real
+       lead screw turns out *slower* than the 0.15 policy cap, then it is the
+       cap or the mechanism that needs revisiting — not this property quietly
+       going back under it. PR6/PR7 own that. -->
+  <xacro:property name="column_lift_effort" value="120.0"/>
+  <xacro:property name="column_lift_velocity" value="0.25"/>
+  <!-- Derived, so that retuning any property above moves the whole column
+       instead of leaving one number behind. -->
+  <!-- Height of the rail's bottom face above `base_link`, m: the chassis
+       puck's top surface, computed from `base.xacro`'s own properties rather
+       than transcribed as 0.115. Rooting the mast at `base_link` (z = 0, axle
+       height) would bury its lower 115 mm inside the chassis solid — the D29
+       chassis/wheel bug again — and hardcoding the sum would leave the column
+       behind the next time the puck moves. -->
+  <xacro:property name="column_base_z" value="${chassis_z_offset + chassis_height / 2}"/>
+  <xacro:property name="column_travel" value="${max_column_height - min_column_height}"/>
+  <!-- The mast spans the travel *plus* the carriage it carries: at full
+       extension the carriage's top face must still be on the rail, not past the
+       end of it. -->
+  <xacro:property name="column_rail_length"
+                  value="${column_travel + column_carriage_height + column_rail_overtravel}"/>
+  <!-- The rail's collision/visual box is centred in its own link frame, so the
+       link frame sits half a rail above the bottom face. -->
+  <xacro:property name="column_rail_joint_z" value="${column_base_z + column_rail_length / 2}"/>
+  <!-- `column_lift`'s origin, in the rail's frame: the height the mount datum
+       sits at when the joint is at its *lower* limit, i.e. carriage resting on
+       the bottom of the rail with its top face one carriage-height up. Written
+       as "the datum's height in base_link, minus the rail frame's" so the
+       intent survives a retune of either. -->
+  <xacro:property name="column_lift_origin_z"
+                  value="${column_base_z + column_carriage_height - min_column_height
+                           - column_rail_joint_z}"/>
+  <!-- ==================================================================
+       Geometry
+       ================================================================== -->
+  <!-- The static mast. `base_link` (the root frame, declared in
+       robot.urdf.xacro) carries no geometry; the rail hangs off it exactly as
+       the chassis does. -->
+  <joint name="column_rail_joint" type="fixed">
+    <parent link="base_link"/>
+    <child link="column_rail_link"/>
+    <origin xyz="0 0 ${column_rail_joint_z}" rpy="0 0 0"/>
+  </joint>
+  <link name="column_rail_link">
+    <visual>
+      <geometry>
+        <box size="${column_rail_width} ${column_rail_depth} ${column_rail_length}"/>
+      </geometry>
+    </visual>
+    <collision>
+      <geometry>
+        <box size="${column_rail_width} ${column_rail_depth} ${column_rail_length}"/>
+      </geometry>
+    </collision>
+    <inertial>
+      <mass value="${column_rail_mass}"/>
+      <!-- Solid box about its own centre. -->
+      <inertia
+        ixx="${column_rail_mass * (column_rail_depth * column_rail_depth
+                                   + column_rail_length * column_rail_length) / 12}"
+        iyy="${column_rail_mass * (column_rail_width * column_rail_width
+                                   + column_rail_length * column_rail_length) / 12}"
+        izz="${column_rail_mass * (column_rail_width * column_rail_width
+                                   + column_rail_depth * column_rail_depth) / 12}"
+        ixy="0" ixz="0" iyz="0"/>
+    </inertial>
+  </link>
+  <!-- The lift itself: one prismatic joint, one STS3215 (D26). The axis is
+       written `0 0 1` under an identity rpy, so it is +z in the rail's frame
+       and — the rail joint being axis-aligned too — +z in `base_link`. It is
+       the *composition* that has to come out vertical, which is what the gate
+       asserts (D29's lesson applied to the column: a lift that travels sideways
+       satisfies "prismatic, limits 0.00-1.20" perfectly). -->
+  <joint name="column_lift" type="prismatic">
+    <parent link="column_rail_link"/>
+    <child link="column_top"/>
+    <origin xyz="0 0 ${column_lift_origin_z}" rpy="0 0 0"/>
+    <axis xyz="0 0 1"/>
+    <limit lower="${min_column_height}" upper="${max_column_height}"
+           effort="${column_lift_effort}" velocity="${column_lift_velocity}"/>
+  </joint>
+  <!-- The carriage. Its link frame origin is the **mount datum** — the top
+       face of the plate — so everything PR3.5/PR4 hang off `column_top` is
+       placed relative to a surface rather than to the middle of a solid. The
+       body itself therefore sits entirely below that origin, which is what the
+       -height/2 offsets say, and is why this link's shape is deliberately *not*
+       readable with the identity-origin helper the base's shapes use. -->
+  <link name="column_top">
+    <visual>
+      <origin xyz="0 0 ${-column_carriage_height / 2}" rpy="0 0 0"/>
+      <geometry>
+        <box size="${column_carriage_width} ${column_carriage_depth} ${column_carriage_height}"/>
+      </geometry>
+    </visual>
+    <collision>
+      <origin xyz="0 0 ${-column_carriage_height / 2}" rpy="0 0 0"/>
+      <geometry>
+        <box size="${column_carriage_width} ${column_carriage_depth} ${column_carriage_height}"/>
+      </geometry>
+    </collision>
+    <inertial>
+      <origin xyz="0 0 ${-column_carriage_height / 2}" rpy="0 0 0"/>
+      <mass value="${column_carriage_mass}"/>
+      <!-- Solid box about its own centre, which is half a carriage below the
+           mount datum: hence the <origin> above, without which the carriage
+           would swing about a point outside itself. -->
+      <inertia
+        ixx="${column_carriage_mass * (column_carriage_depth * column_carriage_depth
+                                       + column_carriage_height * column_carriage_height) / 12}"
+        iyy="${column_carriage_mass * (column_carriage_width * column_carriage_width
+                                       + column_carriage_height * column_carriage_height) / 12}"
+        izz="${column_carriage_mass * (column_carriage_width * column_carriage_width
+                                       + column_carriage_depth * column_carriage_depth) / 12}"
+        ixy="0" ixz="0" iyz="0"/>
+    </inertial>
+  </link>
 </robot>
