Commit message: feat(pr8b): dfki-ric MuJoCo sim bringup green — spawn, controllers, joint command (issue #92)
Swap the MuJoCo sim from ros-controls/mujoco_ros2_control to dfki-ric's
implementation (jazzy, f151b7d) which embeds its own controller_manager and
loads the MJCF synchronously — resolving the sim-spawn std::bad_alloc that
blocked PR8b.

- robot.repos: dfki-ric/mujoco_ros2_control @ f151b7d (no mujoco_vendor).
- colcon_defaults.yaml: scope BUILD_TESTING=OFF to the vendored core + Release.
- pixi.toml: libglvnd, ros-jazzy-cv-bridge, ros-jazzy-pcl-conversions (R-PR8b-13).
- overlay.xml: actuator types per dfki-ric PRM classifier (wheels <velocity kv>,
  joints <position kp> no dampratio); drop gripper <equality> (neq 2->0; dfki-ric
  reads URDF <mimic> natively); omit <camera> (ncam=0, headless EGL safety).
- URDF ros2_control.xacro: plugin mujoco_ros2_control/MujocoSystem; MJCF path/freq
  are node params; mirror joints state-only.
- mujoco.launch.py: franka pattern — spawners -> /controller_manager, real_time_factor
  key, controllers.yaml as node param, sim start gated spawning (R-PR8b-11/14).
- tests updated for the new model (nu 16->18, neq 2->0, camera->site/ncam) and the
  @_BAD_ALLOC_SKIP removed so the ACCEPTANCE smoke test_joint_command_moves_sim_state
  actually runs.

Gate integrity (finishing): the vendored package's own upstream CTest tests were
regenerated/aggregated into colcon test-result and failed it. Full run now selects
ONLY owned packages and clears vendored result areas:
- scripts/check_test_integrity.py: --packages-select on owned (not --packages-skip);
  new delete_vendored_results() clears vendored test_results/ + CTest Testing/ residues
  (colcon test-result --all has no package filter and CTest Test.xml is not xunit-parsable).
- scripts/tests/test_audit.py: 3 unit tests for delete_vendored_results.

Full `pixi run test` GREEN (838/0/0/0, All stages passed); smoke passed; ratchet raised
_workspace_tooling 189->192, robot_bringup 4->5. status.md details. Not merged.

File: src/robot_description/urdf/robot.urdf.xacro (robot description, xacro)
@@ -31,8 +31,9 @@
   <!-- Root frame of the whole robot. Everything else hangs off this. -->
   <link name="base_link"/>
-  <!-- The MuJoCo hardware-interface block (PR8b). The launch overrides this -->
-  <!-- with the real derived-scene path; see the comment at the top of the file. -->
+  <!-- The MuJoCo hardware-interface block (PR8b). dfki-ric's plugin reads the
+       MJCF path, sim frequency and GUI from NODE parameters (mujoco.launch.py),
+       not from the URDF, so this macro takes no arguments. The mujoco_model_path
+       arg is kept for backwards-compat with any launcher-injected xacro call. -->
   <xacro:arg name="mujoco_model_path" default="/tmp/derived_scene.xml"/>
-  <xacro:sisyphus_mujoco_control
-      mujoco_model_path="$(arg mujoco_model_path)"/>
+  <xacro:sisyphus_mujoco_control/>
 </robot>

File: src/robot_description/urdf/ros2_control.xacro (robot description, xacro)
@@ -3,22 +3,22 @@
   ros2_control hardware interfaces for the Sisyphus robot (PR8b / issue #92).
   The ros2_control tag declares the MuJoCo hardware plugin and the joint
-  interfaces mujoco_ros2_control exposes. The MJCF (overlay.xml + derived
-  pipeline) is the actuator authority; here we name the same actuator per
-  joint and choose the command interface type, per the command-interface to
-  MJCF-actuator-type matrix (R-PR8b-6):
-    velocity command, MJCF intvelocity/velocity actuator, the 3 wheels
-    position command,  MJCF position actuator,  column, arm, driven grippers
-  The 2 gripper-mirror joints are mimics: a mimic param (and NO command
-  interface) tells the plugin to derive their value/command from the driven
-  joint, matching the URDF mimic with multiplier -1.
+  interfaces dfki-ric's mujoco_ros2_control exposes. The MJCF (overlay.xml +
+  derived pipeline) is the actuator authority; here we name the same actuator
+  per joint and choose the command interface type, per the command-interface to
+  MJCF-actuator-type matrix (R-PR8b-6, as adapted for dfki-ric in the probe):
+    velocity command, MJCF <velocity> actuator, the 3 wheels
+    position command,  MJCF <position>  actuator,  column, arm, grippers (+mirrors)
+  dfki-ric's plugin is `MujocoSystem` (NOT ros-controls' MujocoSystemInterface).
+  The MJCF path, sim frequency and GUI are NODE parameters (see
+  mujoco.launch.py), not hardware params. dfki-ric reads URDF <mimic> tags
+  natively (so the gripper mirrors below declare state interfaces only, no
+  command interface); the plugin drives each mirror's own MJCF position
+  actuator from the driven command x -1 (see gripper.xacro <mimic>).
 -->
 <robot xmlns:xacro="http://www.ros.org/wiki/xacro">
-  <xacro:macro name="sisyphus_mujoco_control" params="mujoco_model_path">
+  <xacro:macro name="sisyphus_mujoco_control" params="">
     <ros2_control name="MujocoSystem" type="system">
       <hardware>
-        <plugin>mujoco_ros2_control/MujocoSystemInterface</plugin>
-        <param name="mujoco_model">${mujoco_model_path}</param>
-        <param name="headless">true</param>
-        <param name="sim_speed_factor">1.0</param>
+        <plugin>mujoco_ros2_control/MujocoSystem</plugin>
       </hardware>
       <!-- mobile base, 3 continuous wheels: velocity command -->
@@ -123,9 +123,10 @@
         <state_interface name="effort"/>
       </joint>
-      <!-- gripper mirrors: mimics of the driven joints (R-PR8b-6); no command
-           interface, derived from the drivers. -->
+      <!-- gripper mirrors: mimics of the driven joints, via the URDF <mimic>
+           tag in gripper.xacro (multiplier -1). dfki-ric reads that natively
+           and drives each mirror's own MJCF position actuator from the driven
+           command; so the mirrors declare STATE interfaces only (no command
+           interface), per the dfki-ric franka-hand pattern. -->
       <joint name="left_gripper_mirror">
-        <param name="mimic">left_gripper</param>
-        <param name="multiplier">-1</param>
         <state_interface name="position"/>
         <state_interface name="velocity"/>
@@ -133,6 +134,4 @@
       </joint>
       <joint name="right_gripper_mirror">
-        <param name="mimic">right_gripper</param>
-        <param name="multiplier">-1</param>
         <state_interface name="position"/>
         <state_interface name="velocity"/>
