Commit message: fix(i156): stabilise jaw DOF and negate the mirror jaw's declared limits
The sim's gripper jaws diverged from a clean qpos0=0 within ~25 steps and
jammed on jaw self-contact at +0.39/-0.49 rad, outside the declared
[-1.5, 0] range, so no jaw ever tracked a command and MoveIt refused every
plan with START_STATE_IN_COLLISION.

Two defects in gripper.xacro:

* the jaw DOF is a pure-P (kp=100) loop on ~2e-5 kg*m^2 links at dt=2 ms
  (500 Hz) -- an undamped, numerically unstable oscillator. Add a
  joint-level viscous damping (URDF <dynamics damping=0.5>, MuJoCo
  dof_damping) to all four jaw joints. 0.5 is ~5.5x the joint's critical
  damping (2*sqrt(kp*I) ~= 0.09) and was picked from an executed sweep
  (0.2 -> 4.2 mrad overshoot, 0.3 -> 0.7 mrad, 0.5 -> 1e-5 rad with no
  reverse step). kp stays 100; no actuator dampratio/kv (that would set
  biasprm[2] != 0 and make the joint uncommandable to dfki-ric), no effort
  increase, no mass/geometry change.
* the mirror jaw declared the DRIVEN joint's limits [-1.5, 0] under
  <mimic multiplier='-1'>, so the plugin clamped an 'open' command back to
  0. Its declared limits become the exact negation [0, +1.5].

File: src/robot_description/urdf/gripper.xacro (robot description, xacro)
@@ -107,4 +107,34 @@
   <xacro:property name="gripper_joint_lower" value="-1.5"/>
   <xacro:property name="gripper_joint_upper" value="0.0"/>
+  <!-- Joint-level viscous damping (issue #156, R-M1). The jaw links' inertia
+       is ~2e-5 kg*m^2; the sim's <position kp="100"> actuator is a pure P loop
+       with no velocity term, so at dt=0.002 s (500 Hz) the jaw DOF was an
+       UNSTABLE, undamped high-frequency oscillator: from qpos0=0 with ctrl=0
+       it diverged within ~25 steps and jammed on jaw self-contact at
+       +0.39/-0.49 rad, outside the declared [-1.5, 0] range and the reason
+       MoveIt refused every plan (START_STATE_IN_COLLISION). Measured
+       (drivable model, dt=0.002 s, full-range step command) the damped joint
+       is stable and monotone: 0.2 rad overshoot 4.2 mrad, 0.3 -> 0.7 mrad,
+       0.5 -> 1e-5 rad with 0 reverse steps; the sweep and the rejected
+       `armature` alternative are in the feature's implementation.md. This
+       value is ~5.5x the joint's critical damping (2*sqrt(kp*I) ~= 0.09
+       N*m*s/rad), chosen with margin rather than at the stability edge. It is
+       a JOINT term (MuJoCo `dof_damping`, via URDF <dynamics damping>), NOT an
+       actuator `dampratio`/`kv`: dfki-ric classifies a <position> actuator as
+       POSITION only while biasprm[2] == 0, so an actuator-level velocity gain
+       would make the jaw uncommandable. kp stays 100 (the jaws must stay
+       stiff enough to hold a grasp, #155). -->
+  <xacro:property name="gripper_joint_damping" value="0.5"/>
+  <!-- The mirror jaw's declared limits are the EXACT NEGATION of the driven
+       jaw's (issue #156, R-M2). The mirror is a `<mimic multiplier="-1">`
+       follower, so its reachable set is the driven joint's range reflected
+       through zero: with the driven at [-1.5, 0] the mirror must be [0, +1.5].
+       Giving the mirror the driven joint's own [-1.5, 0] made an "open"
+       command (driven -1.5 -> mirror +1.5) fall outside the mirror's declared
+       range; the dfki-ric plugin then clamps the mirror command to 0
+       (mujoco_system.cpp position branch), so the mirror never opened. Written
+       as `0 - <driven bound>` so the two can never drift apart. -->
+  <xacro:property name="gripper_mirror_lower" value="${0.0 - gripper_joint_upper}"/>
+  <xacro:property name="gripper_mirror_upper" value="${0.0 - gripper_joint_lower}"/>
   <!-- ==================================================================
        The fingertip sub-macro. A single rigid box link with a real
@@ -182,4 +212,5 @@
       <limit lower="${gripper_joint_lower}" upper="${gripper_joint_upper}"
              effort="${gripper_joint_effort}" velocity="${gripper_joint_velocity}"/>
+      <dynamics damping="${gripper_joint_damping}"/>
     </joint>
     <link name="${name}_gripper_upper_jaw_link">
@@ -203,5 +234,7 @@
     <!-- Mirror jaw joint: same +y axis, pivot + lever reflected across the grip
          plane (z -> -z); <mimic multiplier="-1"> makes it follow the driven
-         joint with equal-and-opposite rotation. -->
+         joint with equal-and-opposite rotation. Its <limit> is the negation of
+         the driven joint's (gripper_mirror_lower/upper above), so the -1 mimic
+         never commands it out of range (issue #156, R-M2). -->
     <joint name="${name}_gripper_mirror" type="revolute">
       <parent link="${name}_gripper_base_link"/>
@@ -209,6 +242,7 @@
       <origin xyz="${gripper_pivot_x} ${gripper_tuck} ${-gripper_pivot_z}" rpy="0 0 0"/>
       <axis xyz="0 1 0"/>
-      <limit lower="${gripper_joint_lower}" upper="${gripper_joint_upper}"
+      <limit lower="${gripper_mirror_lower}" upper="${gripper_mirror_upper}"
              effort="${gripper_joint_effort}" velocity="${gripper_joint_velocity}"/>
+      <dynamics damping="${gripper_joint_damping}"/>
       <mimic joint="${name}_gripper" multiplier="-1"/>
     </joint>

Commit message: fix(i156): calibrate the jaw damping to the declared velocity limit
Red-team NOTE 2: `dof_damping` also sets the jaw's slew speed. With the
actuator force clamped to +/-effort (3.0 N*m) and the damping torque -d*qdot,
the terminal speed is v = effort/d, so d = 0.5 measured 6.02 rad/s -- 1.7x the
joint's declared 3.5 rad/s `velocity` limit, with the actuator pinned at its
clamp for the whole slew.

Re-chosen as d = effort/velocity = 3.0/3.5 ~= 0.857 (the speed-matched value)
rounded up to 0.9: measured peak 3.345 rad/s (4.4 % under the declared limit;
the exact 0.857 measured 3.505, 0.15 % over, on the 4-step startup transient).
Stability improves (zeta 2.30 -> 4.14), monotone (max reverse step 3e-6 rad),
no out-of-range excursion, mirror == -driven to 2.2e-16, all four actuators
still POSITION.

Also fixes red-team NOTE 1 (the durable comment's numbers: I_eff 1.18e-4 not
~2e-5, 2*sqrt(kp*I) 0.217 not 0.09, omega 921 not 2.3e3) and NOTE 6 (the
mirror-limit negation is the mimic offset == 0 case).

File: src/robot_description/urdf/gripper.xacro (robot description, xacro)
@@ -107,23 +107,37 @@
   <xacro:property name="gripper_joint_lower" value="-1.5"/>
   <xacro:property name="gripper_joint_upper" value="0.0"/>
-  <!-- Joint-level viscous damping (issue #156, R-M1). The jaw links' inertia
-       is ~2e-5 kg*m^2; the sim's <position kp="100"> actuator is a pure P loop
-       with no velocity term, so at dt=0.002 s (500 Hz) the jaw DOF was an
-       UNSTABLE, undamped high-frequency oscillator: from qpos0=0 with ctrl=0
+  <!-- Joint-level viscous damping (issue #156, R-M1/R-M2). The jaw DOF's
+       EFFECTIVE inertia is I_eff ~= 1.18e-4 kg*m^2 (measured, mj_fullM at
+       qpos0): dominated not by the jaw link's own rotational inertia but by
+       the parallel-axis term of the 0.01 kg fingertip box 0.106 m off the axis
+       (1.13e-4), which a link-inertia-only estimate drops. The sim's
+       <position kp="100"> actuator is a pure P loop with no velocity term, so
+       at dt=0.002 s (500 Hz) the jaw DOF was an UNSTABLE, undamped
+       high-frequency oscillator: undamped omega = sqrt(kp/I) ~= 921 rad/s
+       (omega*dt ~= 1.84, only ~3.4 steps/period), and from qpos0=0 with ctrl=0
        it diverged within ~25 steps and jammed on jaw self-contact at
        +0.39/-0.49 rad, outside the declared [-1.5, 0] range and the reason
        MoveIt refused every plan (START_STATE_IN_COLLISION). Measured
        (drivable model, dt=0.002 s, full-range step command) the damped joint
-       is stable and monotone: 0.2 rad overshoot 4.2 mrad, 0.3 -> 0.7 mrad,
-       0.5 -> 1e-5 rad with 0 reverse steps; the sweep and the rejected
+       is stable and monotone: d=0.2 overshoots the declared limit by 5 mrad,
+       d=0.3 by 0.8 mrad, while d=0.5 and d=0.9 stay inside it (<=4e-5 rad)
+       with <=7e-6 rad maximum reverse step; the sweep and the rejected
        `armature` alternative are in the feature's implementation.md. This
-       value is ~5.5x the joint's critical damping (2*sqrt(kp*I) ~= 0.09
-       N*m*s/rad), chosen with margin rather than at the stability edge. It is
-       a JOINT term (MuJoCo `dof_damping`, via URDF <dynamics damping>), NOT an
-       actuator `dampratio`/`kv`: dfki-ric classifies a <position> actuator as
-       POSITION only while biasprm[2] == 0, so an actuator-level velocity gain
-       would make the jaw uncommandable. kp stays 100 (the jaws must stay
-       stiff enough to hold a grasp, #155). -->
-  <xacro:property name="gripper_joint_damping" value="0.5"/>
+       value is ~4.1x the joint's critical damping (2*sqrt(kp*I) ~= 0.217
+       N*m*s/rad), chosen with margin rather than at the stability edge. `d` is
+       ALSO calibrated against the servo's own declared limits: with the
+       actuator force clamped to +/-gripper_joint_effort and the damping torque
+       -d*qdot, the slew's terminal speed is v_terminal = effort/d, so
+       d = effort/velocity = 3.0/3.5 ~= 0.857 is the speed-matched value for
+       the declared 3.5 rad/s limit; 0.9 is that value rounded up, and it keeps
+       the MEASURED peak (3.34 rad/s) below the declared limit (the exact 0.857
+       measures 3.505 rad/s over the 4-step startup transient). A sim that
+       slews a jaw faster than its declared velocity would be internally
+       inconsistent. It is a JOINT term (MuJoCo `dof_damping`, via URDF
+       <dynamics damping>), NOT an actuator `dampratio`/`kv`: dfki-ric
+       classifies a <position> actuator as POSITION only while biasprm[2] == 0,
+       so an actuator-level velocity gain would make the jaw uncommandable. kp
+       stays 100 (the jaws must stay stiff enough to hold a grasp, #155). -->
+  <xacro:property name="gripper_joint_damping" value="0.9"/>
   <!-- The mirror jaw's declared limits are the EXACT NEGATION of the driven
        jaw's (issue #156, R-M2). The mirror is a `<mimic multiplier="-1">`
@@ -134,5 +148,8 @@
        range; the dfki-ric plugin then clamps the mirror command to 0
        (mujoco_system.cpp position branch), so the mirror never opened. Written
-       as `0 - <driven bound>` so the two can never drift apart. -->
+       as `0 - <driven bound>` so the two can never drift apart. NOTE: this
+       negation is the *offset == 0* case: it holds only while the driven
+       joint's `<mimic>` carries no `offset`; a future `<mimic offset="c">`
+       makes the mirror's reach [c-upper, c-lower] and must revisit this. -->
   <xacro:property name="gripper_mirror_lower" value="${0.0 - gripper_joint_upper}"/>
   <xacro:property name="gripper_mirror_upper" value="${0.0 - gripper_joint_lower}"/>
@@ -236,5 +253,6 @@
          joint with equal-and-opposite rotation. Its <limit> is the negation of
          the driven joint's (gripper_mirror_lower/upper above), so the -1 mimic
-         never commands it out of range (issue #156, R-M2). -->
+         never commands it out of range (issue #156, R-M2). The negation is the
+         `mimic offset == 0` case only; revisit it if an `offset` is added. -->
     <joint name="${name}_gripper_mirror" type="revolute">
       <parent link="${name}_gripper_base_link"/>

Commit message: fix(i156): jaw actuation — stabilise the jaw DOF and negate the mirror jaw's limits (#157)
* fix(i156): stabilise jaw DOF and negate the mirror jaw's declared limits

The sim's gripper jaws diverged from a clean qpos0=0 within ~25 steps and
jammed on jaw self-contact at +0.39/-0.49 rad, outside the declared
[-1.5, 0] range, so no jaw ever tracked a command and MoveIt refused every
plan with START_STATE_IN_COLLISION.

Two defects in gripper.xacro:

* the jaw DOF is a pure-P (kp=100) loop on ~2e-5 kg*m^2 links at dt=2 ms
  (500 Hz) -- an undamped, numerically unstable oscillator. Add a
  joint-level viscous damping (URDF <dynamics damping=0.5>, MuJoCo
  dof_damping) to all four jaw joints. 0.5 is ~5.5x the joint's critical
  damping (2*sqrt(kp*I) ~= 0.09) and was picked from an executed sweep
  (0.2 -> 4.2 mrad overshoot, 0.3 -> 0.7 mrad, 0.5 -> 1e-5 rad with no
  reverse step). kp stays 100; no actuator dampratio/kv (that would set
  biasprm[2] != 0 and make the joint uncommandable to dfki-ric), no effort
  increase, no mass/geometry change.
* the mirror jaw declared the DRIVEN joint's limits [-1.5, 0] under
  <mimic multiplier='-1'>, so the plugin clamped an 'open' command back to
  0. Its declared limits become the exact negation [0, +1.5].

* test(i156): pin the jaw contract in sim, URDF and the derived MJCF

* robot_bringup: test_gripper_jaws_track_a_full_range_command launches the
  real bringup and drives the driven jaws open -> closed -> open through the
  shipped arm_gripper_position_controller, asserting from /joint_states that
  they track (settle within 0.05 rad), move monotonically through interior
  values (a sweep, not a jump), stay inside the declared limits at every
  sample, and that each mirror jaw is the exact negation of its driven jaw.
  Fails on the pre-fix URDF with the issue's own numbers (driven ~+0.41,
  mirror ~-0.49, jammed out of range) and passes after it.
* robot_description: assert the mirror jaw's declared limits are the driven
  joint's negation ([0, +1.5]), carry the same effort/velocity, and that all
  four jaw joints declare the stabilising <dynamics damping> while every jaw
  actuator stays a POSITION actuator with kp=100 (biasprm[2] == 0).
* robot_description: assert the DERIVED MJCF carries the negated mirror range
  (jnt_range [0, 1.5]) and the joint damping.
* robot_bringup: the stale 'left_gripper saturates after ~0.01 of a step'
  comment is now history -- point it at the jaw-tracking test.

* chore(i156): raise the test-count baseline for the grown suites

`pixi run test` will not rewrite the baseline from a red run, so the two
entries this change grows are set by hand to the counts the run produced
(what a green run would write):

* robot_description 83 -> 96 (94 non-linter tests already ran on the base
  commit; this change adds the 2 jaw-contract tests)
* robot_bringup 19 -> 21 (20 already ran; this change adds the jaw-tracking
  smoke)

The file was already drifted on main (robot_description 83 vs 94 produced,
robot_mcp 99 vs 102) because a fully green run is what maintains it and the
MoveIt acceptance test has been red; only the two entries this change touches
are moved here. `pixi run test` is red for two pre-existing, unrelated
reasons (robot_brain's shipped OpenClaw fragment vs the 2026.10.3 CLI it was
provisioned with; a Nav2 timing failure in test_pr3_navigate that reproduces
identically on the pre-fix URDF) -- both recorded in the feature's
implementation.md.

* fix(i156): calibrate the jaw damping to the declared velocity limit

Red-team NOTE 2: `dof_damping` also sets the jaw's slew speed. With the
actuator force clamped to +/-effort (3.0 N*m) and the damping torque -d*qdot,
the terminal speed is v = effort/d, so d = 0.5 measured 6.02 rad/s -- 1.7x the
joint's declared 3.5 rad/s `velocity` limit, with the actuator pinned at its
clamp for the whole slew.

Re-chosen as d = effort/velocity = 3.0/3.5 ~= 0.857 (the speed-matched value)
rounded up to 0.9: measured peak 3.345 rad/s (4.4 % under the declared limit;
the exact 0.857 measured 3.505, 0.15 % over, on the 4-step startup transient).
Stability improves (zeta 2.30 -> 4.14), monotone (max reverse step 3e-6 rad),
no out-of-range excursion, mirror == -driven to 2.2e-16, all four actuators
still POSITION.

Also fixes red-team NOTE 1 (the durable comment's numbers: I_eff 1.18e-4 not
~2e-5, 2*sqrt(kp*I) 0.217 not 0.09, omega 921 not 2.3e3) and NOTE 6 (the
mirror-limit negation is the mimic offset == 0 case).

* test(i156): correct the jaw-inertia number in the damping docstrings

The two damping tests' docstrings repeated the ~2e-5 figure red-team NOTE 1
falsified; the jaw DOF's effective inertia is 1.18e-4 kg*m^2. Comment-only;
also records the mimic offset == 0 assumption at the mirror-negation assert
(NOTE 6). No assertions changed.

File: src/robot_description/urdf/gripper.xacro (robot description, xacro)
@@ -107,4 +107,51 @@
   <xacro:property name="gripper_joint_lower" value="-1.5"/>
   <xacro:property name="gripper_joint_upper" value="0.0"/>
+  <!-- Joint-level viscous damping (issue #156, R-M1/R-M2). The jaw DOF's
+       EFFECTIVE inertia is I_eff ~= 1.18e-4 kg*m^2 (measured, mj_fullM at
+       qpos0): dominated not by the jaw link's own rotational inertia but by
+       the parallel-axis term of the 0.01 kg fingertip box 0.106 m off the axis
+       (1.13e-4), which a link-inertia-only estimate drops. The sim's
+       <position kp="100"> actuator is a pure P loop with no velocity term, so
+       at dt=0.002 s (500 Hz) the jaw DOF was an UNSTABLE, undamped
+       high-frequency oscillator: undamped omega = sqrt(kp/I) ~= 921 rad/s
+       (omega*dt ~= 1.84, only ~3.4 steps/period), and from qpos0=0 with ctrl=0
+       it diverged within ~25 steps and jammed on jaw self-contact at
+       +0.39/-0.49 rad, outside the declared [-1.5, 0] range and the reason
+       MoveIt refused every plan (START_STATE_IN_COLLISION). Measured
+       (drivable model, dt=0.002 s, full-range step command) the damped joint
+       is stable and monotone: d=0.2 overshoots the declared limit by 5 mrad,
+       d=0.3 by 0.8 mrad, while d=0.5 and d=0.9 stay inside it (<=4e-5 rad)
+       with <=7e-6 rad maximum reverse step; the sweep and the rejected
+       `armature` alternative are in the feature's implementation.md. This
+       value is ~4.1x the joint's critical damping (2*sqrt(kp*I) ~= 0.217
+       N*m*s/rad), chosen with margin rather than at the stability edge. `d` is
+       ALSO calibrated against the servo's own declared limits: with the
+       actuator force clamped to +/-gripper_joint_effort and the damping torque
+       -d*qdot, the slew's terminal speed is v_terminal = effort/d, so
+       d = effort/velocity = 3.0/3.5 ~= 0.857 is the speed-matched value for
+       the declared 3.5 rad/s limit; 0.9 is that value rounded up, and it keeps
+       the MEASURED peak (3.34 rad/s) below the declared limit (the exact 0.857
+       measures 3.505 rad/s over the 4-step startup transient). A sim that
+       slews a jaw faster than its declared velocity would be internally
+       inconsistent. It is a JOINT term (MuJoCo `dof_damping`, via URDF
+       <dynamics damping>), NOT an actuator `dampratio`/`kv`: dfki-ric
+       classifies a <position> actuator as POSITION only while biasprm[2] == 0,
+       so an actuator-level velocity gain would make the jaw uncommandable. kp
+       stays 100 (the jaws must stay stiff enough to hold a grasp, #155). -->
+  <xacro:property name="gripper_joint_damping" value="0.9"/>
+  <!-- The mirror jaw's declared limits are the EXACT NEGATION of the driven
+       jaw's (issue #156, R-M2). The mirror is a `<mimic multiplier="-1">`
+       follower, so its reachable set is the driven joint's range reflected
+       through zero: with the driven at [-1.5, 0] the mirror must be [0, +1.5].
+       Giving the mirror the driven joint's own [-1.5, 0] made an "open"
+       command (driven -1.5 -> mirror +1.5) fall outside the mirror's declared
+       range; the dfki-ric plugin then clamps the mirror command to 0
+       (mujoco_system.cpp position branch), so the mirror never opened. Written
+       as `0 - <driven bound>` so the two can never drift apart. NOTE: this
+       negation is the *offset == 0* case: it holds only while the driven
+       joint's `<mimic>` carries no `offset`; a future `<mimic offset="c">`
+       makes the mirror's reach [c-upper, c-lower] and must revisit this. -->
+  <xacro:property name="gripper_mirror_lower" value="${0.0 - gripper_joint_upper}"/>
+  <xacro:property name="gripper_mirror_upper" value="${0.0 - gripper_joint_lower}"/>
   <!-- ==================================================================
        The fingertip sub-macro. A single rigid box link with a real
@@ -182,4 +229,5 @@
       <limit lower="${gripper_joint_lower}" upper="${gripper_joint_upper}"
              effort="${gripper_joint_effort}" velocity="${gripper_joint_velocity}"/>
+      <dynamics damping="${gripper_joint_damping}"/>
     </joint>
     <link name="${name}_gripper_upper_jaw_link">
@@ -203,5 +251,8 @@
     <!-- Mirror jaw joint: same +y axis, pivot + lever reflected across the grip
          plane (z -> -z); <mimic multiplier="-1"> makes it follow the driven
-         joint with equal-and-opposite rotation. -->
+         joint with equal-and-opposite rotation. Its <limit> is the negation of
+         the driven joint's (gripper_mirror_lower/upper above), so the -1 mimic
+         never commands it out of range (issue #156, R-M2). The negation is the
+         `mimic offset == 0` case only; revisit it if an `offset` is added. -->
     <joint name="${name}_gripper_mirror" type="revolute">
       <parent link="${name}_gripper_base_link"/>
@@ -209,6 +260,7 @@
       <origin xyz="${gripper_pivot_x} ${gripper_tuck} ${-gripper_pivot_z}" rpy="0 0 0"/>
       <axis xyz="0 1 0"/>
-      <limit lower="${gripper_joint_lower}" upper="${gripper_joint_upper}"
+      <limit lower="${gripper_mirror_lower}" upper="${gripper_mirror_upper}"
              effort="${gripper_joint_effort}" velocity="${gripper_joint_velocity}"/>
+      <dynamics damping="${gripper_joint_damping}"/>
       <mimic joint="${name}_gripper" multiplier="-1"/>
     </joint>
